File: 2nr9_v2.kicad_pcb (KiCad board)
At the start: 2 copper layers, 116 x 76.4 mm, 22 parts

Commit message: upload v2 pcb
Routing:
- net P15: track 37.4 -> 27.3 mm
- net GND: track 145.6 -> 142.6 mm, vias 22 -> 20
- net P19: track 111.4 -> 109.0 mm, vias 1 -> 2
- net P18: track 77.0 -> 74.7 mm, vias 1 -> 2
- net P16: track 67.1 -> 68.5 mm
- net P20: track 62.4 -> 61.4 mm, vias 1 -> 2
